Commit message: tuning quad setting up setpoint generator and change the mass

File: urdf/camera_multirotor.urdf.xacro (robot description, xacro)
@@ -11,5 +11,5 @@
   <xacro:property name="use_mesh_file" value="true" />
   <xacro:property name="mesh_file" value="model://quadrotor/meshes/quadrotor_base.dae" />
-  <xacro:property name="mass" value="2.856" />
+  <xacro:property name="mass" value="1.4" />
   <xacro:property name="body_width" value="0.4" />
   <xacro:property name="body_height" value="0.225" />
